File: Hardware/CCD_boardRev1/CCD_Board.kicad_pcb (KiCad board)
At the start: 2 copper layers, 46.5 x 30 mm, 12 parts, among them Q1 Q_PNP_ECB, U1 74AHC04, U2 TCD1304

Commit message: Fixed things grant suggested
Routing:
- net +3V3: track 66.5 -> 63.8 mm
Changed lines of the file:
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@@
   (setup
     (pad_to_mask_clearance 0)
+    (aux_axis_origin 85.09 80.01)
     (pcbplotparams
       (layerselection 0x00010fc_ffffffff)
@@
   (gr_arc (start 85.344 53.848) (mid 86.534318 50.974318) (end 89.408 49.784) (layer "Edge.Cuts") (width 0.1))
   (via (at 105.41 73.406) (size 0.8) (drill 0.4) (layers "F.Cu" "B.Cu") (free) (net 1))
+  (segment (start 114.935 54.725) (end 113.405 56.255) (width 0.25) (layer "F.Cu") (net 2))
   (segment (start 116.205 78.04) (end 116.205 77.663249) (width 0.25) (layer "F.Cu") (net 2))
   (segment (start 118.455 76.48) (end 117.561751 76.48) (width 0.25) (layer "F.Cu") (net 2))
   (segment (start 108.966 75.184) (end 108.966 71.882) (width 0.25) (layer "F.Cu") (net 2))
-  (segment (start 101.643278 56.443722) (end 98.397 56.443722) (width 0.25) (layer "F.Cu") (net 2))
+  (segment (start 113.405 56.255) (end 113.216278 56.443722) (width 0.25) (layer "F.Cu") (net 2))
+  (segment (start 112.776 56.896) (end 113.405 56.267) (width 0.25) (layer "F.Cu") (net 2))
   (segment (start 118.745 77.663249) (end 117.561751 76.48) (width 0.25) (layer "F.Cu") (net 2))
+  (segment (start 98.397 56.487) (end 98.806 56.896) (width 0.25) (layer "F.Cu") (net 2))
   (segment (start 118.745 78.04) (end 118.745 77.663249) (width 0.25) (layer "F.Cu") (net 2))
-  (segment (start 113.216278 56.443722) (end 101.643278 56.443722) (width 0.25) (layer "F.Cu") (net 2))
   (segment (start 106.942 68.235) (end 106.942 69.858) (width 0.25) (layer "F.Cu") (net 2))
   (segment (start 108.966 71.882) (end 106.942 69.858) (width 0.25) (layer "F.Cu") (net 2))
@@
   (segment (start 113.665 77.663249) (end 112.481751 76.48) (width 0.25) (layer "F.Cu") (net 2))
   (segment (start 113.665 78.04) (end 113.665 77.663249) (width 0.25) (layer "F.Cu") (net 2))
-  (segment (start 114.935 54.725) (end 113.216278 56.443722) (width 0.25) (layer "F.Cu") (net 2))
   (segment (start 112.481751 76.48) (end 110.49 76.48) (width 0.25) (layer "F.Cu") (net 2))
+  (segment (start 98.806 56.896) (end 112.776 56.896) (width 0.25) (layer "F.Cu") (net 2))
   (segment (start 95.857 59.69) (end 98.397 59.69) (width 0.25) (layer "F.Cu") (net 2))
   (segment (start 115.021751 76.48) (end 112.481751 76.48) (width 0.25) (layer "F.Cu") (net 2))
   (segment (start 110.262 76.48) (end 108.966 75.184) (width 0.25) (layer "F.Cu") (net 2))
+  (segment (start 97.79 55.88) (end 98.397 56.487) (width 0.25) (layer "F.Cu") (net 2))
+  (segment (start 110.49 76.48) (end 110.262 76.48) (width 0.25) (layer "F.Cu") (net 2))
+  (segment (start 117.561751 76.48) (end 115.021751 76.48) (width 0.25) (layer "F.Cu") (net 2))
   (segment (start 97.79 54.8) (end 97.79 55.88) (width 0.25) (layer "F.Cu") (net 2))
-  (segment (start 110.49 76.48) (end 110.262 76.48) (width 0.25) (layer "F.Cu") (net 2))
-  (segment (start 98.397 56.443722) (end 98.397 59.69) (width 0.25) (layer "F.Cu") (net 2))
-  (segment (start 97.79 55.88) (end 98.353722 56.443722) (width 0.25) (layer "F.Cu") (net 2))
-  (segment (start 117.561751 76.48) (end 115.021751 76.48) (width 0.25) (layer "F.Cu") (net 2))
-  (segment (start 98.353722 56.443722) (end 101.643278 56.443722) (width 0.25) (layer "F.Cu") (net 2))
+  (segment (start 113.405 56.267) (end 113.405 56.255) (width 0.25) (layer "F.Cu") (net 2))
+  (segment (start 98.397 56.487) (end 98.397 59.69) (width 0.25) (layer "F.Cu") (net 2))
   (segment (start 120.015 73.09) (end 120.015 69.839852) (width 0.25) (layer "F.Cu") (net 3))
   (segment (start 120.015 69.839852) (end 112.395 62.219852) (width 0.25) (layer "F.Cu") (net 3))
