File: FlourometerBoard_Hardware/FlourometerBoard_Hardware.kicad_sch (KiCad schematic)
At the start: 13 parts, among them J1 RJ45_LED_Shielded, U1 Teensy4.1_DEV-16771, U3 OKI

Commit message: Added 5V to LED connectors
Also added FETs to LEDs on breakout.
Parts:
- removed Conn3: Molex_SL_05, MRDT_Connectors:MOLEX_SL_05_Vertical, symbol MRDT_Connectors:Molex_SL_05
- added Conn3: Molex_SL_07, MRDT_Connectors:MOLEX_SL_07_Vertical, symbol MRDT_Connectors:Molex_SL_07
Connections:
- net +5V: now also Conn3.5
- net 400nm LED: now also Conn3.4
- net 430nm LED: now also Conn3.3
- net 522nm LED: now also Conn3.2
- net 530nm LED: now also Conn3.1
- net GND: now also Conn3.6, Conn3.7
Changed lines of the file:
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@@
   (junction (at 119.38 86.36) (diameter 0) (color 0 0 0 0)
+  )
+  (junction (at 167.64 34.29) (diameter 0) (color 0 0 0 0)
   )
   (junction (at 74.93 124.46) (diameter 0) (color 0 0 0 0)
@@
     (stroke (width 0) (type default))
   )
+  (wire (pts (xy 165.1 34.29) (xy 167.64 34.29))
+    (stroke (width 0) (type default))
+  )
   (wire (pts (xy 69.85 124.46) (xy 74.93 124.46))
     (stroke (width 0) (type default))
@@
     (stroke (width 0) (type default))
   )
+  (wire (pts (xy 167.64 31.75) (xy 167.64 34.29))
+    (stroke (width 0) (type default))
+  )
   (wire (pts (xy 105.41 25.4) (xy 105.41 27.94))
     (stroke (width 0) (type default))
@@
     (stroke (width 0) (type default))
   )
+  (wire (pts (xy 162.56 38.1) (xy 166.37 38.1))
+    (stroke (width 0) (type default))
+  )
   (wire (pts (xy 101.6 96.52) (xy 127 96.52))
     (stroke (width 0) (type default))
@@
     (stroke (width 0) (type default))
   )
-  (wire (pts (xy 162.56 31.75) (xy 166.37 31.75))
-    (stroke (width 0) (type default))
-  )
   (wire (pts (xy 26.67 114.3) (xy 29.21 114.3))
     (stroke (width 0) (type default))
@@
     (stroke (width 0) (type default))
   )
+  (wire (pts (xy 167.64 34.29) (xy 170.18 34.29))
+    (stroke (width 0) (type default))
+  )
   (wire (pts (xy 132.08 43.18) (xy 132.08 44.45))
     (stroke (width 0) (type default))
@@
     (stroke (width 0) (type default))
   )
+  (wire (pts (xy 165.1 34.29) (xy 165.1 31.75))
+    (stroke (width 0) (type default))
+  )
   (wire (pts (xy 26.67 111.76) (xy 29.21 111.76))
     (stroke (width 0) (type default))
@@
   )
   (wire (pts (xy 22.86 101.6) (xy 29.21 101.6))
+    (stroke (width 0) (type default))
+  )
+  (wire (pts (xy 162.56 31.75) (xy 162.56 38.1))
     (stroke (width 0) (type default))
   )
@@
     (property "Intersheetrefs" "${INTERSHEET_REFS}" (at 154.94 48.1607 90)
       (effects (font (size 1.27 1.27)) (justify right) hide)
-    )
-  )
-  (symbol (lib_id "MRDT_Connectors:Molex_SL_05") (at 163.83 26.67 90) (unit 1)
-    (in_bom yes) (on_board yes) (dnp no) (fields_autoplaced)
-    (property "Reference" "Conn3" (at 157.48 19.05 90)
-      (effects (font (size 1.524 1.524)))
-    )
-    (property "Value" "Molex_SL_05" (at 157.48 21.59 90)
-      (effects (font (size 1.524 1.524)))
-    )
-    (property "Footprint" "MRDT_Connectors:MOLEX_SL_05_Vertical" (at 163.83 26.67 0)
-      (effects (font (size 1.524 1.524)) hide)
-    )
-    (property "Datasheet" "" (at 163.83 26.67 0)
-      (effects (font (size 1.524 1.524)) hide)
-    )
-    (pin "1")
-    (pin "2")
-    (pin "3")
-    (pin "4")
-    (pin "5")
-    (instances
-      (project "FlourometerBoard_Hardware"
-        (path "/b4982880-e7f7-4cba-b3f5-03d53d819057"
-          (reference "Conn3") (unit 1)
-        )
-      )
     )
   )
@@
     )
   )
-  (symbol (lib_id "power:GND") (at 166.37 31.75 0) (unit 1)
-    (in_bom yes) (on_board yes) (dnp no) (fields_autoplaced)
-    (property "Reference" "#PWR010" (at 166.37 38.1 0)
-      (effects (font (size 1.27 1.27)) hide)
-    )
-    (property "Value" "GND" (at 166.37 36.83 0)
-      (effects (font (size 1.27 1.27)))
-    )
-    (property "Footprint" "" (at 166.37 31.75 0)
-      (effects (font (size 1.27 1.27)) hide)
-    )
-    (property "Datasheet" "" (at 166.37 31.75 0)
+  (symbol (lib_id "power:GND") (at 170.18 34.29 0) (unit 1)
+    (in_bom yes) (on_board yes) (dnp no) (fields_autoplaced)
+    (property "Reference" "#PWR010" (at 170.18 40.64 0)
+      (effects (font (size 1.27 1.27)) hide)
+    )
+    (property "Value" "GND" (at 170.18 39.37 0)
+      (effects (font (size 1.27 1.27)))
+    )
+    (property "Footprint" "" (at 170.18 34.29 0)
+      (effects (font (size 1.27 1.27)) hide)
+    )
+    (property "Datasheet" "" (at 170.18 34.29 0)
       (effects (font (size 1.27 1.27)) hide)
     )
@@
     )
   )
-  (symbol (lib_id "power:GND") (at 132.08 44.45 0) (unit 1)
-    (in_bom yes) (on_board yes) (dnp no) (fields_autoplaced)
-    (property "Reference" "#PWR016" (at 132.08 50.8 0)
-      (effects (font (size 1.27 1.27)) hide)
-    )
-    (property "Value" "GND" (at 132.08 49.53 0)
-      (effects (font (size 1.27 1.27)))
-    )
-    (property "Footprint" "" (at 132.08 44.45 0)
-      (effects (font (size 1.27 1.27)) hide)
-    )
-    (property "Datasheet" "" (at 132.08 44.45 0)
-      (effects (font (size 1.27 1.27)) hide)
-    )
-    (pin "1")
-    (instances
-      (project "FlourometerBoard_Hardware"
-        (path "/b4982880-e7f7-4cba-b3f5-03d53d819057"
-          (reference "#PWR016") (unit 1)
-        )
-      )
-    )
-  )
-  (symbol (lib_id "Device:C") (at 124.46 86.36 270) (unit 1)
-    (in_bom yes) (on_board yes) (dnp no) (fields_autoplaced)
-    (property "Reference" "C1" (at 124.46 78.74 90)
-      (effects (font (size 1.27 1.27)))
-    )
-    (property "Value" "0.1 uF" (at 124.46 81.28 90)
-      (effects (font (size 1.27 1.27)))
-    )
-    (property "Footprint" "Capacitor_SMD:C_0603_1608Metric_Pad1.08x0.95mm_HandSolder" (at 120.65 87.3252 0)
-      (effects (font (size 1.27 1.27)) hide)
-    )
-    (property "Datasheet" "~" (at 124.46 86.36 0)
-      (effects (font (size 1.27 1.27)) hide)
-    )
-    (pin "1")
-    (pin "2")
-    (instances
-      (project "FlourometerBoard_Hardware"
-        (path "/b4982880-e7f7-4cba-b3f5-03d53d819057"
-          (reference "C1") (unit 1)
-        )
-      )
-    )
-  )
-  (symbol (lib_id "MRDT_Connectors:AndersonPP") (at 167.64 74.93 270) (unit 1)
-    (in_bom yes) (on_board yes) (dnp no) (fields_autoplaced)
-    (property "Reference" "Conn1" (at 173.99 76.2 90)
-      (effects (font (size 1.524 1.524)) (justify left))
-    )
-    (property "Value" "AndersonPP" (at 173.99 78.74 90)
-      (effects (font (size 1.524 1.524)) (justify left))
-    )
-    (property "Footprint" "MRDT_Connectors:Square_Anderson_2_H_Side_By_Side_PV" (at 153.67 71.12 0)
+  (symbol (lib_id "MRDT_Connectors:Molex_SL_07") (at 168.91 26.67 90) (unit 1)
+    (in_bom yes) (on_board yes) (dnp no) (fields_autoplaced)
+    (property "Reference" "Conn3" (at 160.02 19.05 90)
+      (effects (font (size 1.524 1.524)))
+    )
+    (property "Value" "Molex_SL_07" (at 160.02 21.59 90)
+      (effects (font (size 1.524 1.524)))
+    )
+    (property "Footprint" "MRDT_Connectors:MOLEX_SL_07_Vertical" (at 163.83 26.67 0)
       (effects (font (size 1.524 1.524)) hide)
     )
-    (property "Datasheet" "" (at 153.67 71.12 0)
+    (property "Datasheet" "" (at 163.83 26.67 0)
       (effects (font (size 1.524 1.524)) hide)
     )
@@
     (pin "3")
     (pin "4")
+    (pin "5")
+    (pin "6")
+    (pin "7")
+    (instances
+      (project "FlourometerBoard_Hardware"
+        (path "/b4982880-e7f7-4cba-b3f5-03d53d819057"
+          (reference "Conn3") (unit 1)
+        )
+      )
+    )
+  )
+  (symbol (lib_id "power:GND") (at 132.08 44.45 0) (unit 1)
+    (in_bom yes) (on_board yes) (dnp no) (fields_autoplaced)
+    (property "Reference" "#PWR016" (at 132.08 50.8 0)
+      (effects (font (size 1.27 1.27)) hide)
+    )
+    (property "Value" "GND" (at 132.08 49.53 0)
+      (effects (font (size 1.27 1.27)))
+    )
+    (property "Footprint" "" (at 132.08 44.45 0)
+      (effects (font (size 1.27 1.27)) hide)
+    )
+    (property "Datasheet" "" (at 132.08 44.45 0)
+      (effects (font (size 1.27 1.27)) hide)
+    )
+    (pin "1")
+    (instances
+      (project "FlourometerBoard_Hardware"
+        (path "/b4982880-e7f7-4cba-b3f5-03d53d819057"
+          (reference "#PWR016") (unit 1)
+        )
+      )
+    )
+  )
+  (symbol (lib_id "Device:C") (at 124.46 86.36 270) (unit 1)
+    (in_bom yes) (on_board yes) (dnp no) (fields_autoplaced)
+    (property "Reference" "C1" (at 124.46 78.74 90)
+      (effects (font (size 1.27 1.27)))
+    )
+    (property "Value" "0.1 uF" (at 124.46 81.28 90)
+      (effects (font (size 1.27 1.27)))
+    )
+    (property "Footprint" "Capacitor_SMD:C_0603_1608Metric_Pad1.08x0.95mm_HandSolder" (at 120.65 87.3252 0)
+      (effects (font (size 1.27 1.27)) hide)
+    )
+    (property "Datasheet" "~" (at 124.46 86.36 0)
+      (effects (font (size 1.27 1.27)) hide)
+    )
+    (pin "1")
+    (pin "2")
+    (instances
+      (project "FlourometerBoard_Hardware"
+        (path "/b4982880-e7f7-4cba-b3f5-03d53d819057"
+          (reference "C1") (unit 1)
+        )
+      )
+    )
+  )
+  (symbol (lib_id "MRDT_Connectors:AndersonPP") (at 167.64 74.93 270) (unit 1)
+    (in_bom yes) (on_board yes) (dnp no) (fields_autoplaced)
+    (property "Reference" "Conn1" (at 173.99 76.2 90)
+      (effects (font (size 1.524 1.524)) (justify left))
+    )
+    (property "Value" "AndersonPP" (at 173.99 78.74 90)
+      (effects (font (size 1.524 1.524)) (justify left))
+    )
+    (property "Footprint" "MRDT_Connectors:Square_Anderson_2_H_Side_By_Side_PV" (at 153.67 71.12 0)
+      (effects (font (size 1.524 1.524)) hide)
+    )
+    (property "Datasheet" "" (at 153.67 71.12 0)
+      (effects (font (size 1.524 1.524)) hide)
+    )
+    (pin "1")
+    (pin "2")
+    (pin "3")
+    (pin "4")
     (pin "1")
     (instances
@@
         )
       )
+    )
+  )
+  (symbol (lib_id "power:+5V") (at 166.37 38.1 0) (unit 1)
+    (in_bom yes) (on_board yes) (dnp no) (fields_autoplaced)
+    (property "Reference" "#PWR013" (at 166.37 41.91 0)
+      (effects (font (size 1.27 1.27)) hide)
+    )
+    (property "Value" "+5V" (at 166.37 33.02 0)
+      (effects (font (size 1.27 1.27)))
+    )
+    (property "Footprint" "" (at 166.37 38.1 0)
+      (effects (font (size 1.27 1.27)) hide)
+    )
+    (property "Datasheet" "" (at 166.37 38.1 0)
+      (effects (font (size 1.27 1.27)) hide)
+    )
+    (pin "1")
+    (instances
+      (project "FlourometerBoard_Hardware"
+        (path "/b4982880-e7f7-4cba-b3f5-03d53d819057"
+          (reference "#PWR013") (unit 1)
+        )
+      )
