File: FlourometerBoard_Hardware/FlourometerBoard_Hardware.kicad_pcb (KiCad board)
At the start: 2 copper layers, 105.7 x 36.6 mm, 15 parts, among them J1 RJ45_LED_Shielded, U1 Teensy4.1_DEV-16771, U3 OKI

Commit message: Created Gerber Files
Parts:
- added G***: LOGO, MRDT_Silkscreens:0_MRDT_Logo_7.5mm, F.Cu at (95.9, 94.6)
